File: KiCAD/MASTER/MASTER.sch (KiCad schematic (older format))
At the start: 221 parts, among them J1 AudioJack2_Switch, J10 SW CTRL1, J11 AudioJack2_Switch, J12 AudioJack2_Switch, J13 AudioJack2_Switch, J14 AudioJack2_Switch, J15 AudioJack2_Switch, J16 AudioJack2_Switch, J17 AudioJack2_Switch, J18 AudioJack2_Switch, J19 From Preamp, J2 AudioJack2_Switch, J20 SW_CTRL2, J22 Front Input, J23 To Poweramp, J3 AudioJack2_Switch, J30 To Pedal, J31 MIDI IN, J32 MIDI OUT, J4 AudioJack2_Switch, J5 AudioJack2_Switch, J6 AudioJack2_Switch, J7 AudioJack2_Switch, J8 AudioJack2_Switch, J9 To Preamp, Q1 ZVN3306A, Q10 ZVN3306A, Q11 ZVN3306A, Q12 ZVN3306A, Q2 ZVN3306A, Q3 ZVN3306A, Q4 ZVN3306A, Q5 ZVN3306A, Q6 ZVN3306A, Q7 ZVN3306A, Q8 ZVN3306A, Q9 ZVN3306A

Commit message: Master Schematic: Updated input circuit. Added Mute circuit.
Parts:
- removed C?: 10μ, symbol Device:CP
- removed C? (x4): 100n, symbol Device:C
- removed R? (x6): 100, symbol Device:R
- removed R? (x3): 2,2M, symbol Device:R
- removed R? (x2): 100k, symbol Device:R
- removed R?: 10k, symbol Device:R
- removed R?: 27k, symbol Device:R
- removed U? (x6): RC4558, symbol Amplifier_Operational:RC4558
- added C? (x3): 100n, symbol Device:C
- added C?: 10μ, symbol Device:CP
- added C?: 10n, symbol Device:C
- added D?: 1N4148, Diode_THT:D_DO-35_SOD27_P7.62mm_Horizontal, symbol Diode:1N4148
- added J?: Thru Out, symbol Connector:AudioJack2_Switch
- added Q? (x3): ZVN3306A, Package_TO_SOT_THT:TO-92Flat, symbol EDN-symbol:ZVN3306A
- added R? (x2): 2,2M, symbol Device:R
- added R?: 27k, symbol Device:R
- added R? (x2): 10k, symbol Device:R
- added U? (x3): RC4558, symbol Amplifier_Operational:RC4558
- R?: value 4,7k -> 8,2k
Connections:
- net +12V: now also C?.1, U?.8 (V+)
- net +5V: now also R?.1
- net GND: now also C?.2, C?.2, J?.S, Q?.3 (S), Q?.3 (S), Q?.3 (S), R?.2, R?.2, U?.4 (V-); no longer U?.11, U?.13
- net Tuner_signal: now also U?.10; no longer R?.1, U?.7
- net at U?.1, U?.2 (-): now also C?.1, C?.2
- net at R?.1, U?.3 (+), U?.5 (+): now also C?.1, U?.3 (+), U?.5 (+)
- net Mute_signal: now reaches U?.5 (PB4)
- net Mute_signal: now also U?.13, Q?.2 (G), Q?.2 (G)
- net at U?.6 (-), U?.7: now also C?.2, C?.1
- net at U?.12: now also Q?.2 (G)
- net at R?.1, RL1.4 (COM1): now also C?.2, C?.1, Q?.1 (D); no longer C?.1, C?.1
- net at C?.2, D?.1 (K), D?.2 (A)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: now also R?.2; no longer R?.1
- net at C?.1, R?.1, R?.2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: now also R?.1; no longer R?.2
- net at J22.T: now also RL?.8 (NC1), RL?.9 (NC2)
- net at J?21.T: now also RL?.11 (NO2), RL?.6 (NO1)
- net at RL?.13 (COM2), RL?.4 (COM1): now also C?.2, R?.1; no longer C?.2, C?.2
- net at R?.2, U?.5 (+): now also R?.1
- net at U?.6 (-): now also R?.1
- net at C?.1, R?.1, U?.1: now also R?.2
- net at C?.1, R?.1, R?.2: now also Q?.1 (D)
- net at C?.2: now also U?.1, U?.2 (-), U?.6 (-), U?.7
- net at R?.1, R?.2: now also R?.2
- new net: C?.1, D?.2 (A), R?.2, U?.11
- new net: C?.1, C?.2, J?.T, Q?.1 (D), R?.1
- new net: D?.1 (K), R?.1, U?.7
- no-connect marks 56 -> 55
Other:
- moved on the sheet: C?, D?, J22, J30, J?, J?21, Q?, R?, RL?A, RL?B, U?A, U?B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
