File: KiCAD/EDN_Rack_LoopController/Main_board.sch (KiCad schematic (older format))
At the start: 82 parts, among them J30 To Pedal, U1 ATmega324PA-PU

Commit message: Schematic polish, added complete schematic pdf.
Parts:
- added F1, F2: Fuse, symbol Device:Fuse
- gave numbers to parts that had none: 57
Connections:
- net VDC: now also F1.2; no longer D41.1 (K), D42.1 (K)
- net at T1.1 (AA): now also F2.2; no longer SW9.4
- new net: D41.1 (K), D42.1 (K), F1.1
- new net: F2.1, SW9.4
Other:
- moved on the sheet: C1, C2, C23, C24, C25, C26, C27, C28, C29, C3, C30, C31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
